File: hardware/ToF-Module.sch (EAGLE design)
At the start: 25 parts, among them CON1 JST-03, CON2 JST-03, U1 ATMEGA328P, U2 BSS138DWQ, U3 MIC5504_2.8YM5, X1 RESONATOR8M00

Commit message: PCB: first version
Parts:
- removed R1, R2, R3, R4, R5, R6, R7: 10k, resistor:R-EU_R0603
- added RN1, RN2: 10k, resistor-dil:4R-NCAT16
- C1, C2: value 1µF -> 4.7µF
- C5: value 4.7µF -> 0.1µF
- C6: value 0.1µF -> 10µF; device resistor:C-EUC0603 -> resistor:C-EUC0805
- renumbered TP1 to SDA, TP2 to SCL, TP3 to EN, TP4 to IRQ
Connections:
- net +2V8: now also RN1A.2, RN1B.2, RN1C.2, RN1D.2; no longer R1.2, R2.2, R3.2, R4.2
- net IRQ: now also RN1D.1; no longer R4.1
- net N$3: now also RN1B.1; no longer R1.1
- net N$4: now also RN1A.1; no longer R2.1
- net RESET: now also RN2C.1; no longer R7.2
- net SCL: now also RN2A.1; no longer R6.1
- net SDA: now also RN2B.1; no longer R5.1
- net VIN: now also RN2A.2, RN2B.2, RN2C.2; no longer R5.2, R6.2, R7.1
- net XSHUT: now also RN1C.1; no longer R3.1

Commit message: hardware: add pullup for ext IRQ line + debug pads
Parts:
- added DEBUG_A, DEBUG_B, DEBUG_C, DEBUG_D: PTR1TP15R, testpad:PTR1TP15R
Connections:
- new net N$1: DEBUG_A.TP, U1.PD6(AIN0)
- new net N$2: DEBUG_B.TP, U1.PD7(AIN1)
- new net N$7: DEBUG_C.TP, U1.PB0(ICP)
- new net N$8: DEBUG_D.TP, U1.PB1(OC1A)
- net +2V8: now also RN2D.1
- net EXT_IRQ: now also RN2D.2
